Commit message: 发布 RM65B 分阶段仿真基线与独立 RViz 操作面板
纳入已验收的公共感知、场景同步、任务候选与执行契约；整理 README 接口速查和完整工作流指南。新增可增量安装的 RViz 面板，保留原生 Plan/Execute，精简界面并验证实际仿真控制链。排除生成目录、日志和上游工作树，供下一阶段实机迁移核验。

File: src/realman_rm65/robot_gazebo/urdf/rm65b_ctm2f110_gz.urdf.xacro (robot description, xacro)
@@ -3,12 +3,16 @@
   <xacro:arg name="pick_place_attachment" default="false"/>
   <xacro:arg name="physical_grasp" default="false"/>
+  <xacro:arg name="wrist_camera" default="true"/>
+  <xacro:arg name="wrist_camera_sensor" default="true"/>
   <xacro:include filename="$(find robot_realman_moveit_config)/urdf/rm65b_ctm2f110.urdf.xacro"/>
   <link name="world"/>
-  <joint name="world_to_rm65b" type="fixed"><parent link="world"/><child link="base_link"/></joint>
+  <!-- Low pedestal reference: the robot base is 0.15 m above world ground. -->
+  <joint name="world_to_rm65b" type="fixed"><parent link="world"/><child link="base_link"/><origin xyz="0 0 0.15" rpy="0 0 0"/></joint>
   <xacro:if value="$(arg wrist_camera)">
+    <xacro:if value="$(arg wrist_camera_sensor)">
     <gazebo reference="wrist_camera_link">
       <sensor name="wrist_rgbd" type="rgbd_camera">
-        <!-- Gazebo camera +X maps to flange +Z. -->
-        <pose>0 0 0 0 -1.57079632679 0</pose>
+        <!-- Keep the image upright when Link6 +Z points toward the object. -->
+        <pose>0 0 0 -1.57079632679 -1.57079632679 0</pose>
         <always_on>true</always_on><update_rate>15</update_rate>
         <topic>/pick_place/rgbd</topic>
@@ -20,4 +24,5 @@
       </sensor>
     </gazebo>
+    </xacro:if>
   </xacro:if>
   <ros2_control name="RM65BCTM2F110GazeboSystem" type="system">
@@ -90,10 +95,10 @@
   </xacro:if>
   <xacro:if value="$(arg physical_grasp)">
-    <!-- Contact-only variant: higher pad friction, no detachable joint. -->
+    <!-- Contact-only variant: moderate pad friction, no detachable joint. -->
     <gazebo reference="ctm2f110_left_pad">
-      <mu1>4.0</mu1><mu2>4.0</mu2>
+      <mu1>1.2</mu1><mu2>1.2</mu2>
     </gazebo>
     <gazebo reference="ctm2f110_right_pad">
-      <mu1>4.0</mu1><mu2>4.0</mu2>
+      <mu1>1.2</mu1><mu2>1.2</mu2>
     </gazebo>
   </xacro:if>

File: src/realman_rm65/robot_gazebo/urdf/rm65b_gz.urdf.xacro (robot description, xacro)
@@ -7,4 +7,5 @@
     <parent link="world"/>
     <child link="base_link"/>
+    <origin xyz="0 0 0.15" rpy="0 0 0"/>
   </joint>
   <ros2_control name="RM65BGazeboSystem" type="system">

File: src/realman_rm65/robot_realman_moveit_config/urdf/rm65b_ctm2f110.urdf.xacro (robot description, xacro)
@@ -1,5 +1,5 @@
 <?xml version="1.0"?>
 <robot xmlns:xacro="http://www.ros.org/wiki/xacro" name="rm_65_description">
-  <xacro:arg name="wrist_camera" default="false"/>
+  <xacro:arg name="wrist_camera" default="true"/>
   <xacro:include filename="$(find rm_description)/urdf/rm_65.urdf.xacro"/>
   <xacro:include filename="$(find robot_changingtek_description)/urdf/ctm2f110.urdf.xacro"/>
@@ -9,14 +9,18 @@
     <link name="wrist_camera_link">
       <inertial><mass value="0.03"/><inertia ixx="0.000003" ixy="0" ixz="0" iyy="0.000003" iyz="0" izz="0.000005"/></inertial>
-      <visual><geometry><cylinder radius="0.018" length="0.006"/></geometry><material name="camera_black"><color rgba="0.1 0.1 0.1 1"/></material></visual>
+      <!-- Simplified RealSense body: width 100 mm, height 30 mm, thickness 20 mm. -->
+      <visual><geometry><box size="0.10 0.02 0.03"/></geometry><material name="camera_black"><color rgba="0.1 0.1 0.1 1"/></material></visual>
+      <collision><geometry><box size="0.10 0.02 0.03"/></geometry></collision>
     </link>
     <joint name="wrist_camera_mount" type="fixed">
       <parent link="Link6"/><child link="wrist_camera_link"/>
-      <origin xyz="0 0 0.10" rpy="0 0 0"/>
+      <!-- Link6 +Y maps to world +Z in the horizontal-forward observation pose. -->
+      <origin xyz="0 0.10 0" rpy="0 0 0"/>
     </joint>
     <link name="camera_color_optical_frame"/>
     <joint name="wrist_camera_optical_joint" type="fixed">
       <parent link="wrist_camera_link"/><child link="camera_color_optical_frame"/>
-      <origin xyz="0 0 0" rpy="0 0 -1.57079632679"/>
+      <!-- Sensor roll correction plus Gazebo-camera to ROS-optical axes. -->
+      <origin xyz="0 0 0" rpy="0 0 3.14159265359"/>
     </joint>
   </xacro:if>
